File: tiny-tesla.kicad_pcb (KiCad board)
At the start: 2 copper layers, 76 x 76 mm, 4 parts

Commit message: Marked the access cutouts
Other:
- board text added: "Access Cutout"
Changed lines of the file:
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@@
     (links 0)
     (no_connects 0)
-    (area 102.907143 61.924999 194.552858 138.075001)
+    (area 102.907143 61.899999 194.552858 138.100001)
     (thickness 1.6)
-    (drawings 1)
+    (drawings 5)
     (tracks 0)
     (zones 0)
@@
     (pad 1 thru_hole circle (at 0 0) (size 5.5 5.5) (drill 3.2) (layers *.Cu *.Mask F.SilkS))
   )
+  (gr_text "Access Cutout" (at 102.5 95.5) (layer Cmts.User)
+    (effects (font (size 1.5 1.5) (thickness 0.3)))
+  )
+  (gr_text "Access Cutout" (at 186.5 128) (layer Cmts.User)
+    (effects (font (size 1.5 1.5) (thickness 0.3)))
+  )
+  (gr_arc (start 150 100) (end 112.467843 105.94451) (angle 33) (layer Dwgs.User) (width 0.2))
+  (gr_arc (start 150 100) (end 184.714727 115.455992) (angle 33) (layer Dwgs.User) (width 0.2))
   (gr_circle (center 150 100) (end 150 138) (layer Edge.Cuts) (width 0.15))
 )
